Commit message: tn-dev branch reinkopiert

File: data/assets/urdf/robot.urdf (robot description, URDF)
Before this commit: robot ur10e_cell, 42 links, 41 joints
Links:
- link left_inner_knuckle: geometry visual mesh filename=../meshes/robotiq-2f140/visual/robotiq_arg2f_140_inner_knuc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
- link right_inner_knuckle: mass None -> 0.0271177346495152; geometry visual mesh filename=../meshes/robotiq-2f140/visual/robotiq_arg2f_140_inner_knuc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
Joints:
- joint left_inner_knuckle_joint: origin xyz=0 -0.0127 0.06142 rpy=2.057963267948966 0 0.0 -> xyz=0 -0.0127 0.06142 rpy=2.357963267948966 0 0.0; type fixed -> revolute
- joint right_inner_knuckle_joint: origin xyz=0 0.0127 0.06142 rpy=2.057963267948966 0 -3.141592653589793 -> xyz=0 0.0127 0.06142 rpy=2.357963267948966 0 -3.141592653589793; type fixed -> revolute
